Commit message: add gripper

File: source/robot_lab/data/Robots/go2_x5/go2_x5.urdf (robot description, URDF)
Before this commit: robot go2_x5, 50 links, 49 joints
Links:
- added link arm_link7, mass 0.064798; collision mesh filename=./meshes/X5/link7.STL; visual mesh filename=./meshes/X5/link7.STL
- added link arm_link8, mass 0.064798; collision mesh filename=./meshes/X5/link8.STL; visual mesh filename=./meshes/X5/link8.STL
- link arm_base_link: mass 0.428 -> 0.43995
- link arm_link1: mass 0.064 -> 0.066982
- link arm_link2: mass 1.165 -> 1.0795
- link arm_link3: mass 0.546 -> 0.54534; geometry collision mesh filename=./meshes/X5/link3.STL; visual mesh filename=./meshes/X5/link3.STL
- link arm_link4: mass 0.080971 -> 0.11714; geometry collision mesh filename=./meshes/X5/link4.STL; visual mesh filename=./meshes/X5/link4.STL
- link arm_link5: mass 0.655 -> 0.63488; geometry collision mesh filename=./meshes/X5/link5.STL; visual mesh filename=./meshes/X5/link5.STL
- link arm_link6: mass 0.581000 -> 0.44089
Joints:
- added joint arm_joint7: type prismatic, parent arm_link6, child arm_link7, origin xyz=0.08657 0.024896 -0.0002436 rpy=0 0 0, axis 0 1 0, limit lower=0 upper=0.044 effort=20 velocity=1
- added joint arm_joint8: type prismatic, parent arm_link6, child arm_link8, origin xyz=0.08657 -0.0249 -0.00024366 rpy=0 0 0, axis 0 -1 0, limit lower=0 upper=0.044 effort=20 velocity=1
- joint arm_gripper_fixed_joint: origin xyz=0.145 0.0 0.0 rpy=0 0 0 -> xyz=0.08657 0.0 0.0 rpy=0 0 0
- joint arm_joint1: origin xyz=0 0 0.0603 rpy=0 0 0 -> xyz=0 0 0.0605 rpy=0 0 0
- joint arm_joint2: origin xyz=0.02 0 0.0402 rpy=0 0 0 -> xyz=0.02 0 0.04 rpy=0 0 0
- joint arm_joint3: origin xyz=-0.264 0 0 rpy=-3.1416 0 0 -> xyz=-0.264 0 0 rpy=3.1416 0 0
- joint arm_joint5: origin xyz=0.06575 -0.001 -0.0825 rpy=0 0 0 -> xyz=0.06775 0.0005 -0.0865 rpy=0 0 0
- joint arm_joint6: origin xyz=0.02845 0 0.0825 rpy=-3.1416 0 0 -> xyz=0.02895 0 0.0865 rpy=-3.1416 0 0
